Commit message: Add build log for sjtu_drone_interfaces package installation and compilation

File: install/sjtu_drone_description/share/sjtu_drone_description/urdf/sjtu_drone.urdf.xacro (robot description, xacro)
@@ -4,6 +4,10 @@
   <!-- Need argument to get from launch file -->
   <xacro:arg name="params_path" default="$(find sjtu_drone_bringup)/config/drone.yaml"/>
+  <xacro:arg name="takeoff_hover_height" default="-1.0"/>
+  <xacro:arg name="takeoff_vertical_speed" default="-1.0"/>
   <!-- Need seperate property for xacro inorder processing -->
   <xacro:property name="params_path" value="$(arg params_path)"/>
+  <xacro:property name="takeoff_hover_height_arg" value="$(arg takeoff_hover_height)"/>
+  <xacro:property name="takeoff_vertical_speed_arg" value="$(arg takeoff_vertical_speed)"/>
   <!-- Read in the yaml dict as mp (short for model parameters) -->
   <xacro:property name="mp" value="${xacro.load_yaml(params_path)}"/>
@@ -94,4 +98,6 @@
       <motionDriftNoise>${mp['motionDriftNoise']}</motionDriftNoise>
       <motionDriftNoiseTime>${mp['motionDriftNoiseTime']}</motionDriftNoiseTime>
+      <takeoffHoverHeight>${float(takeoff_hover_height_arg) if float(takeoff_hover_height_arg) >= 0.0 else mp['takeoffHoverHeight']}</takeoffHoverHeight>
+      <takeoffVerticalSpeed>${float(takeoff_vertical_speed_arg) if float(takeoff_vertical_speed_arg) > 0.0 else mp['takeoffVerticalSpeed']}</takeoffVerticalSpeed>
     </plugin>
   </gazebo>

Commit message: Refactor code structure for improved readability and maintainability

File: install/sjtu_drone_description/share/sjtu_drone_description/urdf/sjtu_drone.urdf.xacro (robot description, xacro)
@@ -1,292 +1 @@
-<?xml version="1.0" ?>
-<robot name="sjtu_drone" xmlns:xacro="http://www.ros.org/wiki/xacro">
-<!-- https://answers.ros.org/question/379014/passing-outside-parameters-into-urdf-file-using-xacro/ -->
-  <!-- Need argument to get from launch file -->
-  <xacro:arg name="params_path" default="$(find sjtu_drone_bringup)/config/drone.yaml"/>
-  <xacro:arg name="takeoff_hover_height" default="-1.0"/>
-  <xacro:arg name="takeoff_vertical_speed" default="-1.0"/>
-  <!-- Need seperate property for xacro inorder processing -->
-  <xacro:property name="params_path" value="$(arg params_path)"/>
-  <xacro:property name="takeoff_hover_height_arg" value="$(arg takeoff_hover_height)"/>
-  <xacro:property name="takeoff_vertical_speed_arg" value="$(arg takeoff_vertical_speed)"/>
-  <!-- Read in the yaml dict as mp (short for model parameters) -->
-  <xacro:property name="mp" value="${xacro.load_yaml(params_path)}"/>
-  <xacro:property name="M_PI" value="3.14159265359" />
-  <link name="base_footprint"/>
-  <joint name="base_footprint_joint" type="fixed">
-    <origin rpy="0 0 0" xyz="0 0 0"/>
-    <parent link="base_footprint"/>
-    <child link="base_link"/>
-  </joint>
-  <link name="base_link">
-    <inertial>
-      <mass value="1.477"/>
-      <origin rpy="0 0 0" xyz="0 0 0"/>
-      <inertia ixx="0.1152" ixy="0" ixz="0" iyy="0.1152" iyz="0" izz="0.218"/>
-    </inertial>
-    <collision name="sjtu_drone_collision">
-      <origin rpy="0 0 0" xyz="0   0   0.04"/>
-      <geometry>
-        <mesh filename="file://$(find sjtu_drone_description)/models/sjtu_drone/quadrotor_4.stl"/>
-        <!-- <mesh filename="package://sjtu_drone/quadrotor_4.stl"/> -->
-      </geometry>
-    </collision>
-    <visual name="sjtu_drone_visual">
-      <origin rpy="0 0 0" xyz="0   0   0.04"/>
-      <geometry>
-        <mesh filename="file://$(find sjtu_drone_description)/models/sjtu_drone/quadrotor_4.dae"/>
-        <!-- <mesh filename="package://sjtu_drone/quadrotor_4.dae"/> -->
-      </geometry>
-    </visual>
-  </link>
-  <joint name="sonar_joint" type="fixed">
-    <parent link="base_link" />
-    <child link="sonar_link" />
-    <origin rpy="0 ${M_PI/2} 0" xyz="0 0 0"/>
-  </joint>
-  <link name="sonar_link"/>
-  <joint name="front_cam_joint" type="fixed">
-    <origin rpy="0 0 0" xyz="0.2 0 0"/>
-    <parent link="base_link" />
-    <child link="front_cam_link" />
-  </joint>
-  <link name="front_cam_link"/>
-  <joint name="bottom_cam_joint" type="fixed">
-    <origin rpy="0 ${M_PI/2} 0" xyz="0 0 0"/>
-    <parent link="base_link" />
-    <child link="bottom_cam_link" />
-  </joint>
-  <link name="bottom_cam_link"/>
-  <gazebo>
-    <plugin name='simple_drone' filename='libplugin_drone.so'>
-      <ros>
-        <namespace>${mp['namespace']}</namespace>
-        <remapping>cmd_vel:=cmd_vel</remapping>
-        <remapping>imu:=imu</remapping>
-        <remapping>sonar:=sonar</remapping>
-        <remapping>camera_front:=camera_front</remapping>
-        <remapping>camera_bottom:=camera_bottom</remapping>
-        <remapping>camera_front_info:=camera_front_info</remapping>
-        <remapping>camera_bottom_info:=camera_bottom_info</remapping>
-        <remapping>gps:=gps</remapping>
-      </ros>
-      <bodyName>base_link</bodyName>
-      <pub_odom>true</pub_odom>
-      <rollpitchProportionalGain>${mp['rollpitchProportionalGain']}</rollpitchProportionalGain>
-      <rollpitchDifferentialGain>${mp['rollpitchDifferentialGain']}</rollpitchDifferentialGain>
-      <rollpitchLimit>${mp['rollpitchLimit']}</rollpitchLimit>
-      <yawProportionalGain>${mp['yawProportionalGain']}</yawProportionalGain>
-      <yawDifferentialGain>${mp['yawDifferentialGain']}</yawDifferentialGain>
-      <yawLimit>${mp['yawLimit']}</yawLimit>
-      <velocityXYProportionalGain>${mp['velocityXYProportionalGain']}</velocityXYProportionalGain>
-      <velocityXYDifferentialGain>${mp['velocityXYDifferentialGain']}</velocityXYDifferentialGain>
-      <velocityXYLimit>${mp['velocityXYLimit']}</velocityXYLimit>
-      <velocityZProportionalGain>${mp['velocityZProportionalGain']}</velocityZProportionalGain>
-      <velocityZIntegralGain>${mp['velocityZIntegralGain']}</velocityZIntegralGain>
-      <velocityZDifferentialGain>${mp['velocityZDifferentialGain']}</velocityZDifferentialGain>
-      <velocityZLimit>${mp['velocityZLimit']}</velocityZLimit>
-      <positionXYProportionalGain>${mp['positionXYProportionalGain']}</positionXYProportionalGain>
-      <positionXYDifferentialGain>${mp['positionXYDifferentialGain']}</positionXYDifferentialGain>
-      <positionXYIntegralGain>${mp['positionXYIntegralGain']}</positionXYIntegralGain>
-      <positionXYLimit>${mp['positionXYLimit']}</positionXYLimit>
-      <positionZProportionalGain>${mp['positionZProportionalGain']}</positionZProportionalGain>
-      <positionZDifferentialGain>${mp['positionZDifferentialGain']}</positionZDifferentialGain>
-      <positionZIntegralGain>${mp['positionZIntegralGain']}</positionZIntegralGain>
-      <positionZLimit>${mp['positionZLimit']}</positionZLimit>
-      <maxForce>${mp['maxForce']}</maxForce>
-      <motionSmallNoise>${mp['motionSmallNoise']}</motionSmallNoise>
-      <motionDriftNoise>${mp['motionDriftNoise']}</motionDriftNoise>
-      <motionDriftNoiseTime>${mp['motionDriftNoiseTime']}</motionDriftNoiseTime>
-      <takeoffHoverHeight>${float(takeoff_hover_height_arg) if float(takeoff_hover_height_arg) >= 0.0 else mp['takeoffHoverHeight']}</takeoffHoverHeight>
-      <takeoffVerticalSpeed>${float(takeoff_vertical_speed_arg) if float(takeoff_vertical_speed_arg) > 0.0 else mp['takeoffVerticalSpeed']}</takeoffVerticalSpeed>
-    </plugin>
-  </gazebo>
-  <!-- Sensors -->
-  <!-- IMU sensor in 100fps -->
-  <gazebo reference="base_link">
-    <sensor name='sensor_imu' type='imu'>
-      <always_on> 1 </always_on>
-      <visualize>1</visualize>
-      <update_rate> 100 </update_rate>
-      <pose> 0 0 0 0 0 0 </pose>
-      <imu>
-        <noise>
-          <type>gaussian</type>
-          <rate>
-            <mean> 0 </mean>
-            <stddev> 0.01 </stddev>
-          </rate>
-          <accel>
-            <mean> 0 </mean>
-            <stddev> 0.01 </stddev>
-          </accel>
-        </noise>
-      </imu>
-      <plugin name='imu' filename='libgazebo_ros_imu_sensor.so'>
-        <ros>
-          <namespace>${mp['namespace']}</namespace>
-          <!-- <remapping>imu:=imu</remapping> -->
-        </ros>
-        <initial_orientation_as_reference>false</initial_orientation_as_reference>
-        <frame_name>${mp['namespace']}/base_link</frame_name>
-      </plugin>
-    </sensor>
-  </gazebo>
-  <!-- Sonar sensor in 100fps -->
-  <gazebo reference="sonar_link">
-    <sensor name="sonar" type="ray">
-      <always_on>1</always_on>
-      <visualize>1</visualize>
-      <update_rate>30</update_rate>
-      <ray>
-        <scan>
-          <horizontal>
-            <samples>5</samples>
-            <resolution>1.000000</resolution>
-            <min_angle>-0.12</min_angle>
-            <max_angle>0.12</max_angle>
-          </horizontal>
-          <vertical>
-            <samples>5</samples>
-            <resolution>1.000000</resolution>
-            <min_angle>-0.12</min_angle>
-            <max_angle>0.12</max_angle>
-          </vertical>
-        </scan>
-        <range>
-          <min>0.02</min>
-          <max>10</max>
-          <resolution>0.01</resolution>
-        </range>
-        <noise>
-          <type>gaussian</type>
-          <mean>0.0</mean>
-          <stddev>0.01</stddev>
-        </noise>
-      </ray>
-      <plugin name="sonar" filename="libgazebo_ros_ray_sensor.so">
-        <ros>
-          <namespace>${mp['namespace']}</namespace>
-          <!-- <remapping>~/out:=sonar</remapping> -->
-        </ros>
-        <frame_name>${mp['namespace']}/sonar_link</frame_name>
-        <output_type>sensor_msgs/Range</output_type>
-        <radiation_type>ultrasound</radiation_type>
-      </plugin>
-    </sensor>
-  </gazebo>
-  <gazebo reference="front_cam_link">
-    <sensor name="front_camera" type="camera">
-      <always_on>1</always_on>
-      <visualize>1</visualize>
-      <update_rate>60</update_rate>
-      <camera>
-        <horizontal_fov>2.09</horizontal_fov>
-        <image>
-          <width>640</width>
-          <height>360</height>
-          <format>R8G8B8</format>
-        </image>
-        <clip>
-          <near>0.1</near>
-          <far>100</far>
-        </clip>
-        <noise>
-          <type>gaussian</type>
-          <mean>0.0</mean>
-          <stddev>0.01</stddev>
-        </noise>
-      </camera>
-      <plugin name="camera_front" filename="libgazebo_ros_camera.so">
-        <ros>
-          <namespace>${mp['namespace']}</namespace>
-          <!-- <remapping>~/image_raw:=camera_front</remapping>
-          <remapping>~/camera_info:=camera_front_info</remapping> -->
-        </ros>
-        <frame_name>${mp['namespace']}/front_cam_link</frame_name>
-        <camera_name>front</camera_name>
-        <hack_baseline>0.07</hack_baseline>
-      </plugin>
-    </sensor>
-  </gazebo>
-  <!-- downward looking camera -->
-  <gazebo reference="bottom_cam_link">
-    <sensor name="down_camera" type="camera">
-      <always_on>1</always_on>
-      <visualize>1</visualize>
-      <update_rate>15</update_rate>
-      <camera>
-        <horizontal_fov>1.047</horizontal_fov>
-        <image>
-          <width>640</width>
-          <height>360</height>
-          <format>R8G8B8</format>
-        </image>
-        <clip>
-          <near>0.1</near>
-          <far>100</far>
-        </clip>
-        <noise>
-          <type>gaussian</type>
-          <mean>0.0</mean>
-          <stddev>0.01</stddev>
-        </noise>
-      </camera>
-      <plugin name="camera_bottom" filename="libgazebo_ros_camera.so">
-        <ros>
-          <namespace>${mp['namespace']}</namespace>
-          <!-- <remapping>image_raw:=camera_bottom</remapping>
-          <remapping>camera_info:=camera_bottom_info</remapping> -->
-        </ros>
-        <frame_name>${mp['namespace']}/bottom_cam_link</frame_name>
-        <camera_name>bottom</camera_name>
-        <hack_baseline>0.07</hack_baseline>
-      </plugin>
-    </sensor>
-  </gazebo>
-  <gazebo reference="base_link">
-    <sensor name="gps" type="gps">
-      <always_on>1</always_on>
-      <update_rate>30</update_rate>
-      <gps>
-        <position_sensing>
-          <horizontal>
-            <noise type="gaussian">
-              <mean>0.0</mean>
-              <stddev>2e-4</stddev>
-            </noise>
-          </horizontal>
-          <vertical>
-            <noise type="gaussian">
-              <mean>0.0</mean>
-              <stddev>2e-4</stddev>
-            </noise>
-          </vertical>
-        </position_sensing>
-      </gps>
-      <plugin name="gps" filename="libgazebo_ros_gps_sensor.so">
-        <ros>
-          <namespace>${mp['namespace']}</namespace>
-          <remapping>~/out:=~/nav</remapping>
-        </ros>
-        <frame_name>${mp['namespace']}/base_link</frame_name>
-      </plugin>
-    </sensor>
-  </gazebo>
-  <gazebo reference="base_link">
-    <sensor name="collision_sensor" type="contact">
-      <update_rate>100.0</update_rate>
-      <always_on>true</always_on>
-      <contact>
-        <collision>base_footprint_fixed_joint_lump__sjtu_drone_collision_collision</collision>
-      </contact>
-      <plugin name="collision_plugin" filename="libgazebo_ros_bumper.so">
-        <ros>
-          <namespace>${mp['namespace']}</namespace>
-          <!-- <remapping>bumper_states:=bumper_states</remapping> -->
-        </ros>
-        <frame_name>${mp['namespace']}/base_link</frame_name>
-      </plugin>
-    </sensor>
-  </gazebo>
-</robot>
+/home/j/INCSL/IICC26_ws/src/sjtu_drone-ros2/sjtu_drone_description/urdf/sjtu_drone.urdf.xacro
